File: files/kicad/ampcontrol-f103.sch (KiCad schematic (older format))
At the start: 2 parts, among them J1 Conn_LCD, U1 STM32F103CBTx

Commit message: Updated schematics
Parts:
- added C1, C2: 6p2, symbol Device:C
- added C3, C4: 20p, symbol Device:C
- added R1, R2, R3, R4, R5, R6, R7, R8: 1k, symbol Device:R
- added R10, R9: 4k7, symbol Device:R
- added Y1: 32768, symbol Device:Crystal_Small
- added Y2: 8MHz, symbol Device:Crystal_Small
Connections:
- net labels added: +5V, BOOT0, BOOT1, BTN_0, BTN_1, BTN_2, BTN_3, BTN_4, BTN_5, ENC_A, ENC_B, IR, LEFT, MUTE, RIGHT, RX, SCK, SCL, SDA, STBY, SWCLK, SWDIO, TX, USB_DM, USB_DP
- wire segments 54 -> 106
Other:
- moved on the sheet: U1
