File: files/kicad/amp-ili9341/ampcontrol-f103.kicad_pcb (KiCad board)
At the start: 2 copper layers, 94.4 x 64.8 mm, 2 parts, among them J1 Conn_LCD, U1 STM32F103CBTx

Commit message: Add TDA7313 schematic
Connections:
- net /DB10 renamed Net-(J1-Pad9)
- net /DB11 renamed Net-(J1-Pad10)
- net /DB12 renamed Net-(J1-Pad11)
- net /DB13 renamed Net-(J1-Pad12)
- net /DB14 renamed Net-(J1-Pad13)
- net /DB15 renamed Net-(J1-Pad14)
- net /DB8 renamed Net-(J1-Pad7)
- net /DB9 renamed Net-(J1-Pad8)
- net Net-(U1-Pad18) renamed /LEFT
- net Net-(U1-Pad19) renamed /RIGHT
- net Net-(U1-Pad20) renamed /BOOT1
- net Net-(U1-Pad21) renamed /SCL
- net Net-(U1-Pad22) renamed /SDA
- net Net-(U1-Pad29) renamed /IR
- net Net-(U1-Pad30) renamed /TX
- net Net-(U1-Pad31) renamed /RX
- net Net-(U1-Pad32) renamed /USB_DM
- net Net-(U1-Pad33) renamed /USB_DP
- net Net-(U1-Pad34) renamed /SWCLK
- net Net-(U1-Pad37) renamed /SWDIO
- net Net-(U1-Pad39) renamed /SCK
- net Net-(U1-Pad44) renamed /BOOT0
- net Net-(U1-Pad45) renamed /MUTE
- net Net-(U1-Pad46) renamed /STBY
- J1 pad 17: /REST -> /RST
- J1 pad 19: /LEDA -> /BCKL
- U1 pad 2: Net-(U1-Pad2) -> /BCKL
- U1 pad 25: Net-(U1-Pad25) -> /SD_CS
- U1 pad 26: Net-(U1-Pad26) -> /SD_CLK
- U1 pad 27: Net-(U1-Pad27) -> /SD_DO
- U1 pad 28: Net-(U1-Pad28) -> /SD_DIN
- U1 pad 38: Net-(U1-Pad38) -> /RST
- U1 pad 40: Net-(U1-Pad40) -> /RD
- U1 pad 41: Net-(U1-Pad41) -> /WR
- U1 pad 42: Net-(U1-Pad42) -> /RS
- U1 pad 43: Net-(U1-Pad43) -> /CS

Commit message: Update schematics
Parts:
- added C1: 6p2, Capacitor_SMD:C_1206_3216Metric, F.Cu at (153.9, 106.7)
- added C2: 6p2, Capacitor_SMD:C_1206_3216Metric, F.Cu at (196.7, 117.9)
- added C3: 20p, Capacitor_SMD:C_1206_3216Metric, F.Cu at (192.1, 106.7)
- added C4: 20p, Capacitor_SMD:C_1206_3216Metric, F.Cu at (200.2, 88.9)
- added C5: 20p, Capacitor_SMD:C_1206_3216Metric, F.Cu at (190.6, 89.4)
- added C6: 20p, Capacitor_SMD:C_1206_3216Metric, F.Cu at (211.2, 106.2)
- added R10: 4k7, Resistor_SMD:R_1206_3216Metric, F.Cu at (169.8, 85.9)
- added R11: 10k, Resistor_SMD:R_1206_3216Metric, F.Cu at (166.5, 101.6)
- added R12: 10k, Resistor_SMD:R_1206_3216Metric, F.Cu at (206.8, 99.6)
- added R13: 22k, Resistor_SMD:R_1206_3216Metric, F.Cu at (179.3, 79.2)
- added R14: 22k, Resistor_SMD:R_1206_3216Metric, F.Cu at (164.7, 87.4)
- added R15: 22k, Resistor_SMD:R_1206_3216Metric, F.Cu at (164.2, 78.7)
- added R16: 22k, Resistor_SMD:R_1206_3216Metric, F.Cu at (158.5, 101.6)
- added R17: 100k, Resistor_SMD:R_1206_3216Metric, F.Cu at (171.2, 94.0)
- added R18: 100k, Resistor_SMD:R_1206_3216Metric, F.Cu at (172.8, 81.3)
- added R9: 4k7, Resistor_SMD:R_1206_3216Metric, F.Cu at (155.4, 95.0)
- added RV1: 22k, Potentiometer_THT:Potentiometer_Piher_PT-6-V_Vertical, F.Cu at (177.8, 89.8)
- added U2: MCP602, Package_SO:SOIC-8_3.9x4.9mm_P1.27mm, F.Cu at (185.8, 97.7)
- added Y1: 32768, Crystal:Crystal_C38-LF_D3.0mm_L8.0mm_Vertical, F.Cu at (164.6, 93.5)
- added Y2: 8MHz, Crystal:Crystal_HC49-4H_Vertical, F.Cu at (151.1, 85.3)
- moved U1 8.12 mm to (178.3, 107.2), turned to 0 degrees
Connections:
- U1 pad 18: /LEFT -> /SP_L
- U1 pad 19: /RIGHT -> /SP_R

Commit message: Update schematic/pinout binaries
Parts:
- removed R10, R9: 4k7, Resistor_SMD:R_1206_3216Metric
- removed R11, R12: 10k, Resistor_SMD:R_1206_3216Metric
- removed R13, R14, R15, R16: 22k, Resistor_SMD:R_1206_3216Metric
- added R1: 10k, Resistor_SMD:R_1206_3216Metric, F.Cu at (180.1, 100.3)
- added R19: 4k7, Resistor_SMD:R_1206_3216Metric, F.Cu at (182.1, 107.2)
- added R2: 10k, Resistor_SMD:R_1206_3216Metric, F.Cu at (177.5, 105.5)
- added R20: 22k, Resistor_SMD:R_1206_3216Metric, F.Cu at (189.3, 99.5)
- added R3: 22k, Resistor_SMD:R_1206_3216Metric, F.Cu at (180.1, 102.6)
- added R4: 22k, Resistor_SMD:R_1206_3216Metric, F.Cu at (186.6, 94.9)
- added R5: 22k, Resistor_SMD:R_1206_3216Metric, F.Cu at (184.7, 97.2)
- added R6: 22k, Resistor_SMD:R_1206_3216Metric, F.Cu at (172.9, 105.5)
- added R7: 100k, Resistor_SMD:R_1206_3216Metric, F.Cu at (184.7, 99.5)
- added R8: 100k, Resistor_SMD:R_1206_3216Metric, F.Cu at (182.1, 104.9)
- C1, C2: value 6p2 -> 20p
- C3, C4: value 20p -> 6p2
- R17: value 100k -> 22k
- R18: value 100k -> 4k7
- U1: value STM32F103CBTx -> MCP602; footprint Package_QFP:LQFP-48_7x7mm_P0.5mm -> Package_SO:SOIC-8_3.9x4.9mm_P1.27mm
- U2: value MCP602 -> STM32F103CBTx; footprint Package_SO:SOIC-8_3.9x4.9mm_P1.27mm -> Package_QFP:LQFP-48_7x7mm_P0.5mm
- moved C6 38.4 mm to (172.9, 107.8)
- moved C2 29.3 mm to (182.0, 92.6)
- moved Y1 23.7 mm to (185.4, 104.9)
- moved C1 23.6 mm to (177.5, 107.8)
- moved R18 22.9 mm to (189.3, 97.2)
- moved C4 22.0 mm to (180.1, 98.0)
- moved U2 21.0 mm to (165.3, 102.4)
- moved R17 15.6 mm to (184.7, 101.7)
- moved C3 15.6 mm to (182.0, 94.9)
- moved Y2 15.4 mm to (163.6, 94.3)
- moved RV1 14.7 mm to (171.7, 103.2)
- moved U1 13.2 mm to (175.9, 94.2)
- moved C5 5.13 mm to (186.6, 92.6)
Connections:
- net Net-(J1-Pad10) renamed /DB11
- net Net-(J1-Pad11) renamed /DB12
- net Net-(J1-Pad12) renamed /DB13
- net Net-(J1-Pad13) renamed /DB14
- net Net-(J1-Pad14) renamed /DB15
- net Net-(J1-Pad7) renamed /DB8
- net Net-(J1-Pad8) renamed /DB9
- net Net-(J1-Pad9) renamed /DB10
- C1 pad 2: GNDD -> Net-(C1-Pad2)
- C2 pad 1: GNDD -> Net-(C2-Pad1)
- C3 pad 1: GNDD -> Net-(C3-Pad1)
- C3 pad 2: Net-(C3-Pad2) -> GNDD
- C5 pad 1: Net-(C5-Pad1) -> GNDD
- C6 pad 1: Net-(C6-Pad1) -> GNDD
- J1 pad 17: /RST -> /NRST
- R17 pad 1: Net-(R11-Pad2) -> +3V3
- R17 pad 2: /SP_L -> /NRST
- R18 pad 1: Net-(R12-Pad2) -> +5V
- R18 pad 2: /SP_R -> /SCL
- RV1 pad 2: Net-(C5-Pad2) -> Net-(C1-Pad2)
- U1 pad 1: Net-(U1-Pad1) -> /SP_L
- U1 pad 2: /BCKL -> Net-(R1-Pad2)
- U1 pad 3: Net-(C2-Pad2) -> Net-(R3-Pad2)
- U1 pad 4: Net-(C1-Pad1) -> (no net)
- U1 pad 5: Net-(C4-Pad2) -> Net-(R5-Pad2)
- U1 pad 6: Net-(C3-Pad2) -> Net-(R2-Pad2)
- U1 pad 7: Net-(R13-Pad2) -> /SP_R
- U1 pad 8: Net-(U1-Pad8) -> (no net)
- U2 pad 1: /SP_L -> Net-(U2-Pad1)
- U2 pad 2: Net-(R11-Pad2) -> /BCKL
- U2 pad 3: Net-(R14-Pad1) -> Net-(C4-Pad2)
- U2 pad 4: (no net) -> Net-(C3-Pad1)
- U2 pad 5: Net-(R15-Pad2) -> Net-(C6-Pad2)
- U2 pad 6: Net-(R12-Pad2) -> Net-(C5-Pad2)
- U2 pad 7: /SP_R -> /NRST
- U2 pad 8: (no net) -> Net-(U2-Pad8)
- Y1 pad 1: Net-(C1-Pad1) -> Net-(C3-Pad1)
- Y1 pad 2: Net-(C2-Pad2) -> Net-(C4-Pad2)
- Y2 pad 1: Net-(C4-Pad2) -> Net-(C6-Pad2)
- Y2 pad 2: Net-(C3-Pad2) -> Net-(C5-Pad2)
