File: files/kicad/amp-ili9341/ampcontrol-f103.sch (KiCad schematic (older format))
At the start: 18 parts, among them J1 Conn_LCD, U1 STM32F103CBTx, Y1 32768, Y2 8MHz

Commit message: Update schematics
Parts:
- added C5, C6: 20p, Capacitor_SMD:C_1206_3216Metric, symbol Device:C
- added R11, R12: 10k, Resistor_SMD:R_1206_3216Metric, symbol Device:R
- added R13, R14, R15, R16: 22k, Resistor_SMD:R_1206_3216Metric, symbol Device:R
- added R17, R18: 100k, Resistor_SMD:R_1206_3216Metric, symbol Device:R
- added RV1: 22k, Potentiometer_THT:Potentiometer_Piher_PT-6-V_Vertical, symbol Device:R_POT
- added RV2: 22k, symbol Device:R_POT
- added U2: MCP602, Package_SO:SOIC-8_3.9x4.9mm_P1.27mm, symbol Amplifier_Operational:MCP602
- C1, C2, C3, C4: footprint (none) -> Capacitor_SMD:C_1206_3216Metric
- R10, R9: footprint (none) -> Resistor_SMD:R_1206_3216Metric
- Y1: footprint (none) -> Crystal:Crystal_C38-LF_D3.0mm_L8.0mm_Vertical
- Y2: footprint (none) -> Crystal:Crystal_HC49-4H_Vertical
Connections:
- net +3V3: now also R13.1, R15.1
- net GNDD: now also R14.2, R16.2, RV1.3, RV2.3
- net at U1.7 (NRST): now also R13.2
- net LEFT renamed SP_L
- net SP_L: now also R17.2, U2.1
- net RIGHT renamed SP_R
- net SP_R: now also R18.2, U2.7
- new net: R11.2, R17.1, U2.2 (-)
- new net: R14.1, U2.3 (+)
- new net: R15.2, R16.1, U2.5 (+)
- new net: R12.2, R18.1, U2.6 (-)
- new net: C5.1, R11.1
- new net: C5.2, RV1.2
- new net: C6.1, R12.1
- new net: C6.2, RV2.2
- new net IN_L: RV1.1
- new net IN_R: RV2.1
Other:
- moved on the sheet: J1, R1, R2, R3, R4, R5, R6, R7, R8

Commit message: Update and fix schematic
Parts:
- added R3: 22k, Resistor_SMD:R_1206_3216Metric, symbol Device:R
- renumbered C5 to C1, C6 to C2, C1 to C3, C2 to C4, C3 to C5, C4 to C6, R11 to R1, R2 to R10, R3 to R11, R4 to R12, R5 to R13, R6 to R14, R7 to R15, R8 to R16, R13 to R17, R9 to R18, R10 to R19, R12 to R2, R14 to R4, R15 to R5, R16 to R6, R17 to R7, R18 to R8, R1 to R9, U2 to U1, U1 to U2
Connections:
- net +3V3: now also R3.1
- net at R4.1, U1.3 (+): now also R3.2

Commit message: Update schematic/pinout binaries
Parts:
- added R20: 22k, Resistor_SMD:R_1206_3216Metric, symbol Device:R
Connections:
- net +3V3: now also R20.1
- net RD: now also R20.2
- net DB11: now reaches J1.10 (Pin_10)
- net DB12: now reaches J1.11 (Pin_11)
- net DB13: now reaches J1.12 (Pin_12)
- net DB14: now reaches J1.13 (Pin_13)
- net DB15: now reaches J1.14 (Pin_14)
- net DB8: now reaches J1.7 (Pin_7)
- net DB9: now reaches J1.8 (Pin_8)
- net DB10: now reaches J1.9 (Pin_9)
- net NRST: now reaches R17.2, U2.7 (NRST)
- net NRST: now also J1.17 (Pin_17)
- net RST renamed HW_RST
- net HW_RST: no longer J1.17 (Pin_17)
Other:
- moved on the sheet: J1

Commit message: Update schematic
Parts:
- added BT1: 3.3V, symbol Device:Battery_Cell
- added C10, C11: 20p, Capacitor_SMD:C_1206_3216Metric, symbol Device:C
- added C12, C9: CP, symbol Device:CP
- added C7: 1.0, Capacitor_SMD:C_1206_3216Metric, symbol Device:C
- added C8: 0.22, Capacitor_SMD:C_1206_3216Metric, symbol Device:C
- added J2: Conn_AUDIO, symbol Connector_Generic:Conn_01x03
- added J3: Conn_USB, symbol Connector_Generic:Conn_01x04
- added J4: Conn_SWD, symbol Connector_Generic:Conn_01x04
- added J5: Conn_BOOT, symbol Connector_Generic:Conn_02x03_Odd_Even
- added R21, R22: 22, Resistor_SMD:R_1206_3216Metric, symbol Device:R
- added R23: 1.5k, Resistor_SMD:R_1206_3216Metric, symbol Device:R
- added R24, R25: 100k, Resistor_SMD:R_1206_3216Metric, symbol Device:R
- added SW1: Reset, symbol Switch:SW_Push
- added U3: AMS1117-3.3, Package_TO_SOT_SMD:SOT-223-3_TabPin2, symbol Regulator_Linear:AMS1117-3.3
- C1, C2: value 20p -> 2.2
- R1, R2: value 10k -> 22k
- R7, R8: value 100k -> 220k
Connections:
- net +3V3: now also C11.2, C12.1, C8.1, J4.1 (Pin_1), J5.1 (Pin_1), J5.2 (Pin_2), U3.2 (VO)
- net +5V: now also C10.2, C9.1, J3.1 (Pin_1), R23.1, U3.3 (VI)
- net BOOT0: now also R24.1
- net BOOT1: now also R25.2
- net GNDD: now also C5.2, C6.2, BT1.2 (-), C10.1, C11.1, C12.2, C7.1, C8.2, C9.2, J2.2 (Pin_2), J3.4 (Pin_4), J4.4 (Pin_4), J5.5 (Pin_5), J5.6 (Pin_6), SW1.2, U3.1 (GND); no longer C5.1, C6.1
- net IN_L: now also J2.1 (Pin_1)
- net IN_R: now also J2.3 (Pin_3)
- net NRST: now also C7.2, SW1.1
- net RD: no longer U2.40 (PB4)
- net SP_L: no longer R7.2, U1.1
- net SWCLK: now also J4.3 (Pin_3)
- net SWDIO: now also J4.2 (Pin_2)
- net USB_DM: now also R21.2
- net USB_DP: now also R22.2, R23.2
- net at U2.1 (VBAT): now also BT1.1 (+)
- new net: C5.1, U2.5 (PD0), Y2.2
- new net: C6.1, U2.6 (PD1), Y2.1
- new net: R7.2, U1.1
- new net: J5.3 (Pin_3), R24.2
- new net: J5.4 (Pin_4), R25.1
- new net: J3.2 (Pin_2), R21.1
- new net: J3.3 (Pin_3), R22.1
Other:
- moved on the sheet: C1, C2, C3, C4, C5, C6, J1, R1, R10, R11, R12, R13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

Commit message: Update project binaries
Connections:
- net GNDD: now also U2.8 (VSSA)
- net SWCLK: now also U2.37 (PA14); no longer U2.34 (PA13)
- net SWDIO: now also U2.34 (PA13); no longer U2.37 (PA14)
Changed lines of the file:
@@
 Text Label 6900 5650 2    50   ~ 0
 SDA
+Text Label 4800 5950 0    50   ~ 0
+SWCLK
 Text Label 4800 5850 0    50   ~ 0
-SWCLK
-Text Label 4800 5950 0    50   ~ 0
 SWDIO
 Wire Wire Line
@@
 	7600 4400 7600 4350
 Wire Wire Line
-	4800 5950 5200 5950
-Wire Wire Line
-	5200 5850 4800 5850
+	4800 5850 5200 5850
+Wire Wire Line
+	5200 5950 4800 5950
 Wire Wire Line
 	900  5550 1200 5550
@@
 Wire Wire Line
 	6500 3950 7600 3950
+Wire Wire Line
+	5700 6250 5700 6350
+Wire Wire Line
+	5700 6350 5800 6350
+Connection ~ 5800 6350
 $EndSCHEMATC
