File: kicad/pwr_33x2/pwr_33x2.kicad_pcb (KiCad board)
At the start: 2 copper layers, 66 x 50.8 mm, 6 parts, among them J1 POW_IN, J2 POW_L, J3 POW_R

Commit message: Move pwr_33x2 to Kicad 6
Other:
- net class Default removed
