File: kicad/tda7313/tda7313.kicad_pcb (KiCad board)
At the start: 2 copper layers, 68.6 x 55.9 mm, 36 parts, among them J1 SP_L, J10 OUT_FL, J11 OUT_RL, J12 OUT_FR, J13 OUT_RR, J14 PWR, J2 IN1_L, J3 IN2_L, J4 IN3_L, J5 IN1_R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

Commit message: Move tda7313 to Kicad 6
Other:
- net class Default removed
