File: kicad/tda7719/tda7719.kicad_pcb (KiCad board)
At the start: 2 copper layers, 63.5 x 38.1 mm, 33 parts, among them J1 IN0, J10 REAR, J11 SUB, J12 PWR, J2 IN4, J3 IN1, J4 IN2, J5 IN5, J6 IN6, J7 I2C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

Commit message: Move tda7719 to Kicad 6
Other:
- net class Default removed
